File: Sense Circuit.kicad_sch (KiCad schematic)
At the start: 0 parts

Commit message: something
Parts:
- added D3: 1N4148, Diode_THT:D_DO-35_SOD27_P7.62mm_Horizontal, symbol Diode:1N4148
- added R3: 50K-100K ohm, symbol Device:R_US
Connections:
- new net From Driver: R3.1
- new net From Sensor: D3.1 (K), R3.2
- new net GND: D3.2 (A)
