File: Drive Circuit.kicad_sch (KiCad schematic)
At the start: 0 parts

Commit message: drive circuit
Parts:
- added Q1: NPN, symbol Simulation_SPICE:NPN
- added R4: 47K/1.1mW, symbol Device:R_US
- added R5: 1K/20mW, symbol Device:R_US
- added R6: 470E/0.47mW, symbol Device:R_US
- added R7: 1K/0.3mW, symbol Device:R_US
Connections:
- new net: Q1.3 (E), R6.1
- new net +12V: R4.1, R5.1
- new net +5V: Q1.1 (C), R5.2
- new net GND: R6.2, R7.2
- new net MCU Square Wave: Q1.2 (B), R4.2, R7.1
